File: hardware/PUTM_EV_AMS_SLAVE_2025.kicad_pcb (KiCad board)
At the start: 4 copper layers, 100 x 23 mm, 147 parts, among them IC2 BQ79616PAPR, J1 M80-5100405, J2 M80-5100405, J4 IDC24, Q2 100V/2W

Commit message: routing 80-90% done
Parts:
- added G***: LOGO, Samacsys:PUTM_Logo_8mm, B.Cu at (176.4, 125.8)
- TH1, TH2: moved to F.Cu
- moved TH2 5.81 mm to (178.9, 121.9), turned to -90 degrees
- moved TH1 5.06 mm to (121.1, 121.9), turned to -90 degrees
Routing:
- net /BQ79616/VC4: track 1.47 -> 87.8 mm, vias 0 -> 4
- net /BQ79616/CB4: track 10.7 -> 93.8 mm, vias 0 -> 3
- net /AUX/TH7+: track 6.06 -> 70.8 mm, vias 0 -> 4
- net /C16+: track 6.02 -> 60.0 mm, vias 0 -> 4
- net /BQ79616/AUX2/TH8+: track 7.00 -> 58.6 mm, vias 0 -> 4
- net /BQ79616/VC8: track 1.47 -> 43.6 mm, vias 0 -> 3
- net /C4+: track 6.02 -> 48.1 mm, vias 0 -> 1
- net /BQ79616/VC5: track 7.76 -> 48.4 mm, vias 0 -> 3
- net /BQ79616/CB3: track 15.4 -> 54.0 mm, vias 0 -> 2
- net /C13+: track 6.02 -> 44.4 mm, vias 0 -> 1
- net /C12+: track 6.02 -> 43.8 mm, vias 0 -> 1
- net /BQ79616/VC3: track 7.76 -> 44.8 mm, vias 0 -> 2
- net /C5+: track 6.02 -> 41.1 mm, vias 0 -> 1
- net /BQ79616/CB5: track 15.4 -> 48.6 mm, vias 0 -> 1
- net /C3+: track 6.02 -> 36.7 mm, vias 0 -> 1
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
Commit message: v2.0.0b done
Routing:
- net /BQ79616/VC12: track 29.9 -> 89.7 mm, vias 2 -> 3
- net /BQ79616/VC13: track 8.13 -> 64.3 mm, vias 0 -> 2
- net /BQ79616/CB12: track 38.4 -> 94.5 mm, vias 2 -> 3
- net /BQ79616/CB13: track 14.0 -> 68.5 mm, vias 0 -> 2
- net /BQ79616/VC14: track 8.13 -> 58.9 mm, vias 0 -> 2
- net /BQ79616/CB14: track 13.7 -> 63.3 mm, vias 0 -> 2
- net /BQ79616/CB15: track 13.8 -> 61.8 mm, vias 0 -> 2
- net /BQ79616/VC15: track 8.07 -> 55.7 mm, vias 0 -> 2
- net /BQ79616/CB16: track 10.4 -> 54.3 mm, vias 0 -> 2
- net /BQ79616/VC16: track 1.48 -> 44.9 mm, vias 0 -> 2
- net /TH1+: track 9.41 -> 34.8 mm, vias 2 -> 1
- net /TH2+: track 11.0 -> 24.9 mm, vias 2 -> 1
- net /BQ79616/VC7: track 33.2 -> 42.2 mm, vias 2 -> 3
- net /BQ79616/VC10: track 33.5 -> 41.8 mm, vias 2 -> 3
- net /BQ79616/CB10: track 35.6 -> 43.4 mm, vias 2 -> 3
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