File: hardware/PUTM_EV_AMS_SLAVE_2025.kicad_pcb (KiCad board)
At the start: 4 copper layers, 100 x 20 mm, 64 parts, among them CN7 4x100nF, IC1 LTC6804HG-1#PBF, J1 TST-110-01-T-D, J2 B02B-PASK-1, J3 B02B-PASK-1, Q1 BCP56

Commit message: sync
Parts:
- removed C18, C19: 100nF, Capacitor_SMD:C_0603_1608Metric
- removed CN7: 4x100nF, Resistor_SMD:R_Array_Convex_4x0603
- removed D21, D23: LED, LED_SMD:LED_0603_1608Metric
- removed R33, R37, R41, R44, R45: 100/1W, Resistor_SMD:R_1210_3225Metric
- removed R34, R38, R42, R46, R48: 330, Resistor_SMD:R_0603_1608Metric
- removed the REF** at (103.5, 113.5)
- removed the REF** at (196.5, 126.5)
- removed RN7: 4x10k, Resistor_SMD:R_Array_Convex_4x0603
- added C9: 100nF, Capacitor_SMD:C_0603_1608Metric, F.Cu at (164.8, 70.8)
- added D11: LED, LED_SMD:LED_0603_1608Metric, F.Cu at (207.9, 69.4)
- added D12: LED, LED_SMD:LED_0603_1608Metric, F.Cu at (189.0, 92.0)
- added R11: 330, Resistor_SMD:R_0603_1608Metric, F.Cu at (205.2, 84.8)
- added R15: 330, Resistor_SMD:R_0603_1608Metric, F.Cu at (215.2, 84.8)
- added R16: 51/2W, Resistor_SMD:R_1206_3216Metric, F.Cu at (216.2, 87.8)
- added R19: 330, Resistor_SMD:R_0603_1608Metric, F.Cu at (189.0, 76.1)
- added R23: 330, Resistor_SMD:R_0603_1608Metric, F.Cu at (191.0, 85.4)
- added R24: 51/2W, Resistor_SMD:R_1206_3216Metric, F.Cu at (190.0, 82.4)
- added R27: 330, Resistor_SMD:R_0603_1608Metric, F.Cu at (191.0, 88.7)
- added R28: 51/2W, Resistor_SMD:R_1206_3216Metric, F.Cu at (190.0, 85.7)
- added R3: 51/2W, Resistor_SMD:R_1206_3216Metric, F.Cu at (190.0, 69.3)
- added R31: 330, Resistor_SMD:R_0603_1608Metric, F.Cu at (191.0, 92.0)
- added R32: 51/2W, Resistor_SMD:R_1206_3216Metric, F.Cu at (190.0, 89.0)
- added RN1: 4x10k, Resistor_SMD:R_Array_Convex_4x0603, F.Cu at (147.9, 73.9)
- C1, C2, C3: value 1uF -> 4.7nF/Y2; footprint Capacitor_SMD:C_0603_1608Metric -> Samacsys:CAPC5728X280N
- C4: value 100nF -> 4.7nF/Y2; footprint Capacitor_SMD:C_0603_1608Metric -> Samacsys:CAPC5728X280N
- C5: value 4.7nF/Y2 -> 100nF; footprint Samacsys:CAPC5728X280N -> Capacitor_SMD:C_0603_1608Metric; moved to F.Cu
- C6, C7, C8: value 4.7nF/Y2 -> 1uF; footprint Samacsys:CAPC5728X280N -> Capacitor_SMD:C_0603_1608Metric; moved to F.Cu
- IC1, Q1, R4: moved to F.Cu
- J1: value TST-110-01-T-D -> M80-5100442; footprint Connector_IDC:IDC-Header_2x10_P2.54mm_Vertical_SMD -> Samacsys:M80-51004YY
- J2: value B02B-PASK-1 -> TST-110-01-T-D; footprint Samacsys:B02BPASK1LFSN -> Connector_IDC:IDC-Header_2x10_P2.54mm_Vertical_SMD; moved to B.Cu
- J3: value B02B-PASK-1 -> M80-5100442; footprint Samacsys:B02BPASK1LFSN -> Samacsys:M80-51004YY
- R1: value 100/1W -> 120; footprint Resistor_SMD:R_1210_3225Metric -> Resistor_SMD:R_0603_1608Metric
- R10, R14, R18, R22, R26, R30: value 330 -> 51/2W; footprint Resistor_SMD:R_0603_1608Metric -> Resistor_SMD:R_1206_3216Metric
- R12, R20: value 120 -> 51/2W; footprint Resistor_SMD:R_0603_1608Metric -> Resistor_SMD:R_1206_3216Metric; moved to F.Cu
- R13, R17, R21, R25, R29, R9: value 100/1W -> 330; footprint Resistor_SMD:R_1210_3225Metric -> Resistor_SMD:R_0603_1608Metric
- R2: value 10k -> 120; moved to F.Cu
- R5: value 100 -> 1k; moved to F.Cu
- R6: value 330 -> 1k
- R7: value 1k -> 100; moved to F.Cu
- R8: value 1k -> 10k; moved to F.Cu
- moved D9 104.0 mm to (204.6, 69.4), turned to 180 degrees
- moved D5 104.0 mm to (222.2, 84.8)
- moved R30 103.0 mm to (210.9, 70.4)
- moved R29 102.8 mm to (207.9, 71.4), turned to 180 degrees
- moved R26 95.0 mm to (207.6, 70.4)
- moved R25 94.8 mm to (204.6, 71.4), turned to 180 degrees
- moved D4 93.8 mm to (217.2, 84.8)
- moved D7 92.0 mm to (201.3, 69.4), turned to 180 degrees
- moved R22 87.1 mm to (204.3, 70.4)
- moved R21 86.9 mm to (201.3, 71.4), turned to 180 degrees
- moved D6 84.1 mm to (191.0, 76.1)
- moved C6 81.1 mm to (164.8, 63.2), turned to 0 degrees
- moved C5 80.0 mm to (164.8, 60.7), turned to 0 degrees
- moved D8 77.4 mm to (189.0, 85.4), turned to -90 degrees
- moved R12 69.8 mm to (206.2, 87.8), turned to 180 degrees
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Connections:
- C1 pad 1: Net-(IC1-VREF2) -> /IN+
- C1 pad 2: /C1- -> /IA+
- C2 pad 1: /L_LTC/VREF2 -> /IN-
- C2 pad 2: /C1- -> /IA-
- C3 pad 1: /L_LTC/VREG -> /IB+
- C3 pad 2: /C1- -> /OUT+
- C4 pad 1: /TH1+ -> /IB-
- C4 pad 2: /C1- -> /OUT-
- C5 pad 1: /IB+ -> /C12+
- C5 pad 2: /OUT+ -> /L_LTC/V-
- C6 pad 1: /IB- -> Net-(IC1-VREF2)
- C6 pad 2: /OUT- -> GND
- C7 pad 1: /IN+ -> /L_LTC/VREF2
- C7 pad 2: /IA+ -> GND
- C8 pad 1: /IN- -> /L_LTC/VREG
- C8 pad 2: /IA- -> GND
- D1 pad 1: /L_LTC/S1 -> /L_LTC/C1
- D10 pad 1: /L_LTC/S10 -> /L_LTC/C10
- D2 pad 1: /L_LTC/S2 -> /L_LTC/C2
- D3 pad 1: /L_LTC/S3 -> /L_LTC/C3
- D4 pad 1: /L_LTC/S4 -> /L_LTC/C4
- D5 pad 1: /L_LTC/S5 -> /L_LTC/C5
- D6 pad 1: /L_LTC/S6 -> /L_LTC/C6
- D7 pad 1: /L_LTC/S7 -> /L_LTC/C7
- D8 pad 1: /L_LTC/S8 -> /L_LTC/C8
- D9 pad 1: /L_LTC/S9 -> /L_LTC/C9
- IC1 pad 10: /C8+ -> /L_LTC/C8
- IC1 pad 11: /L_LTC/S8 -> /L_LTC/C8
- IC1 pad 12: /C7+ -> /L_LTC/C7
- IC1 pad 13: /L_LTC/S7 -> /L_LTC/C7
- IC1 pad 14: /C6+ -> /L_LTC/C6
- IC1 pad 15: /L_LTC/S6 -> /L_LTC/C6
- IC1 pad 16: /C5+ -> /L_LTC/C5
- IC1 pad 17: /L_LTC/S5 -> /L_LTC/C5
- IC1 pad 18: /C4+ -> /L_LTC/C4
- IC1 pad 19: /L_LTC/S4 -> /L_LTC/C4
- IC1 pad 2: /C12+ -> /L_LTC/C12
- IC1 pad 20: /C3+ -> /L_LTC/C3
- IC1 pad 21: /L_LTC/S3 -> /L_LTC/C3
- IC1 pad 22: /C2+ -> /L_LTC/C2
- IC1 pad 23: /L_LTC/S2 -> /L_LTC/C2
- IC1 pad 24: /C1+ -> /L_LTC/C1
- IC1 pad 25: /L_LTC/S1 -> /L_LTC/C1
- IC1 pad 26: /C1- -> /L_LTC/C0
- IC1 pad 3: /L_LTC/S12 -> /L_LTC/C12
- IC1 pad 30: /C1- -> GND
- IC1 pad 31: /C1- -> GND
- IC1 pad 36: /C1- -> GND
- IC1 pad 4: /C11+ -> /L_LTC/C11
- IC1 pad 5: /L_LTC/S11 -> /L_LTC/C11
- IC1 pad 6: /C10+ -> /L_LTC/C10
- IC1 pad 7: /L_LTC/S10 -> /L_LTC/C10
- IC1 pad 8: /C9+ -> /L_LTC/C9
- IC1 pad 9: /L_LTC/S9 -> /L_LTC/C9
- J1 pad 1: /C1- -> /IN+
- J1 pad 2: /C12+ -> /IN-
- J1 pad 3: /C1+ -> unconnected-(J1-Pin_3-Pad3)
- J1 pad 4: /C11+ -> unconnected-(J1-Pin_4-Pad4)
- J2 pad 1: /OUT+ -> GND
- J2 pad 2: /OUT- -> /C12+
- J3 pad 1: /IN+ -> /OUT-
- J3 pad 2: /IN- -> /OUT+
- R1 pad 1: /C11+ -> /IB-
- R1 pad 2: /L_LTC/S11 -> /IB+
- R10 pad 1: /C1+ -> /L_LTC/C1
- R10 pad 2: Net-(D1-A) -> /C1+
- R12 pad 1: /IA+ -> /L_LTC/C2
- R12 pad 2: /IA- -> /C2+
- R13 pad 1: /C2+ -> /C3+
- R13 pad 2: /L_LTC/S2 -> Net-(D3-A)
- R14 pad 1: /C2+ -> /L_LTC/C3
- R14 pad 2: Net-(D2-A) -> /C3+
- R17 pad 1: /C3+ -> /C5+
- R17 pad 2: /L_LTC/S3 -> Net-(D5-A)
- R18 pad 1: /C3+ -> /L_LTC/C5
- R18 pad 2: Net-(D3-A) -> /C5+
- R2 pad 1: /TH1+ -> /IA-
- R2 pad 2: /L_LTC/VREF2 -> /IA+
- R20 pad 1: /IB+ -> /L_LTC/C6
- R20 pad 2: /IB- -> /C6+
- R21 pad 1: /C4+ -> /C7+
- R21 pad 2: /L_LTC/S4 -> Net-(D7-A)
- R22 pad 1: /C4+ -> /L_LTC/C7
- R22 pad 2: Net-(D4-A) -> /C7+
- R25 pad 1: /C5+ -> /C9+
- R25 pad 2: /L_LTC/S5 -> Net-(D9-A)
- R26 pad 1: /C5+ -> /L_LTC/C9
- R26 pad 2: Net-(D5-A) -> /C9+
- R29 pad 1: /C6+ -> /C11+
- R29 pad 2: /L_LTC/S6 -> Net-(D11-A)
- R30 pad 1: /C6+ -> /L_LTC/C11
- R30 pad 2: Net-(D6-A) -> /C11+
- R5 pad 1: /C12+ -> Net-(IC1-IBIAS)
- R5 pad 2: Net-(Q1-C) -> Net-(IC1-ICMP)
- R6 pad 1: /C11+ -> Net-(IC1-ICMP)
- R6 pad 2: Net-(D21-A) -> GND
- R7 pad 1: Net-(IC1-IBIAS) -> /C12+
- R7 pad 2: Net-(IC1-ICMP) -> Net-(Q1-C)
- R8 pad 1: Net-(IC1-ICMP) -> /TH1+
- R8 pad 2: /C1- -> /L_LTC/VREF2
- R9 pad 2: /L_LTC/S1 -> Net-(D1-A)
Routing:
- net /C10+: track 114.8 -> 2.37 mm, vias 1 -> 0
- net /C12+: track 91.1 -> 2.37 mm, vias 3 -> 0
- net /L_LTC/S4: track 69.7 -> 0.00 mm, vias 1 -> 0
- net /L_LTC/S5: track 61.0 -> 0.00 mm, vias 1 -> 0
- net /C9+: track 60.8 -> 2.37 mm, vias 1 -> 0
- net /L_LTC/S12: track 54.7 -> 0.00 mm, vias 3 -> 0
- net /C11+: track 55.8 -> 2.37 mm, vias 3 -> 0
- net /C6+: track 54.0 -> 2.37 mm, vias 1 -> 0
- net /C3+: track 53.1 -> 2.37 mm, vias 1 -> 0
- net /L_LTC/S6: track 50.2 -> 0.00 mm, vias 1 -> 0
- net /IA-: track 49.0 -> 0.00 mm
- net /TH1+: track 48.7 -> 0.00 mm, vias 3 -> 0
- net /L_LTC/S9: track 48.3 -> 0.00 mm, vias 1 -> 0
- net /IA+: track 48.2 -> 0.00 mm
- net /TH2+: track 47.3 -> 0.00 mm, vias 3 -> 0
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- added copper zone on B.Cu, net GND
- added copper zone on F.Cu, net GND
- added copper zone on In1.Cu, net GND
- added copper zone on In2.Cu, net GND
- removed copper zone on B.Cu, net /C1-
- removed copper zone on F.Cu, net /C1-
- removed copper zone on In1.Cu, net /C1-
- removed copper zone on In2.Cu, net /C1-
Other:
- board size 100 x 20 mm -> 100 x 23 mm
- board text removed: "C10"
- board text removed: "C11"
- board text removed: "C12"
- board text removed: "C2"
- board text removed: "C3"
- board text removed: "C4"
- board text removed: "C5"
- board text removed: "C6"
- board text removed: "C7"
- board text removed: "C8"
- board text removed: "C9"
- board text removed: "TMP"

Commit message: rounting + layout
Parts:
- removed RN1: 4x10k, Resistor_SMD:R_Array_Convex_4x0603
- added L1: 100-500uH, Inductor_SMD:L_CommonModeChoke_Coilcraft_1812CAN, B.Cu at (118.0, 116.5)
- added L2: 100-500uH, Inductor_SMD:L_CommonModeChoke_Coilcraft_1812CAN, B.Cu at (182.0, 123.5)
- added R33: 10k, Resistor_SMD:R_0603_1608Metric, F.Cu at (144.0, 112.7)
- added R34: 10k, Resistor_SMD:R_0603_1608Metric, F.Cu at (142.0, 112.7)
- added R35: 10k, Resistor_SMD:R_0603_1608Metric, F.Cu at (144.0, 116.3)
- added R36: 10k, Resistor_SMD:R_0603_1608Metric, F.Cu at (142.0, 116.3)
- moved D5 102.5 mm to (126.7, 122.0)
- moved R17 102.5 mm to (124.8, 122.0)
- moved R18 102.5 mm to (125.8, 125.0)
- moved R22 95.4 mm to (120.8, 116.5), turned to 180 degrees
- moved D4 93.3 mm to (131.7, 122.0)
- moved R15 93.3 mm to (129.8, 122.0)
- moved R16 93.3 mm to (130.8, 125.0)
- moved R21 91.8 mm to (119.8, 113.5), turned to 90 degrees
- moved D7 91.0 mm to (121.7, 113.5), turned to 90 degrees
- moved R26 89.6 mm to (130.8, 116.5), turned to 180 degrees
- moved R25 85.9 mm to (129.8, 113.5), turned to 90 degrees
- moved D9 85.1 mm to (131.7, 113.5), turned to 90 degrees
- moved D6 83.1 mm to (121.8, 122.0)
- moved R19 83.1 mm to (119.8, 122.0)
- moved R20 83.1 mm to (120.8, 125.0)
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Connections:
- C1 pad 2: /IA+ -> /ICL+
- C2 pad 2: /IA- -> /ICL-
- C3 pad 1: /IB+ -> /OCL+
- C4 pad 1: /IB- -> /OCL-
- C5 pad 2: /L_LTC/V- -> GND
Routing:
- net /TH1+: track 0.00 -> 47.4 mm, vias 0 -> 2
- net /TH2+: track 0.00 -> 42.9 mm, vias 0 -> 3
- net /L_LTC/C1: track 2.40 -> 44.8 mm
- net /TH3+: track 0.00 -> 42.2 mm, vias 0 -> 3
- net /L_LTC/C6: track 2.40 -> 37.8 mm, vias 0 -> 2
- net /L_LTC/C0: track 0.00 -> 33.0 mm
- net /C9+: track 2.37 -> 35.0 mm, vias 0 -> 4
- net /L_LTC/C5: track 2.40 -> 33.4 mm, vias 0 -> 2
- net /C3+: track 2.37 -> 32.9 mm, vias 0 -> 1
- net /L_LTC/VREG: track 0.00 -> 30.1 mm
- net /C7+: track 2.37 -> 31.9 mm, vias 0 -> 3
- net /L_LTC/C4: track 2.40 -> 29.1 mm, vias 0 -> 2
- net /C8+: track 2.37 -> 29.0 mm, vias 0 -> 2
- net /L_LTC/C2: track 2.40 -> 27.6 mm
- net /C2+: track 2.37 -> 26.6 mm, vias 0 -> 3
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Other:
- board text added: "C0"
- board text added: "C10"
- board text added: "C11"
- board text added: "C12"
- board text added: "C2"
- board text added: "C3"
- board text added: "C4"
- board text added: "C5"
- board text added: "C6"
- board text added: "C7"
- board text added: "C8"
- board text added: "C9"

Commit message: done
Parts:
- added G***: LOGO, Samacsys:PUTM_Logo_8mm, B.Cu at (174.5, 126.2)
- moved REF** 16.0 mm to (196.5, 128.0)
- moved REF** 16.0 mm to (103.5, 112.0)
- moved C1 7.07 mm to (111.5, 125.5)
- moved C2 7.07 mm to (111.5, 121.5)
- moved C3 7.07 mm to (188.5, 118.5)
- moved C4 7.07 mm to (188.5, 114.5)
- moved L1 7.07 mm to (119.0, 123.5)
- moved L2 7.07 mm to (181.0, 116.5)
- moved J1 7.00 mm to (103.5, 123.5)
- moved J3 7.00 mm to (196.5, 116.5)
- moved R1 2.51 mm to (142.0, 119.8), turned to -90 degrees
Connections:
- net /L_LTC/C0 renamed /LTC/C0
- net /L_LTC/C1 renamed /LTC/C1
- net /L_LTC/C10 renamed /LTC/C10
- net /L_LTC/C11 renamed /LTC/C11
- net /L_LTC/C12 renamed /LTC/C12
- net /L_LTC/C2 renamed /LTC/C2
- net /L_LTC/C3 renamed /LTC/C3
- net /L_LTC/C4 renamed /LTC/C4
- net /L_LTC/C5 renamed /LTC/C5
- net /L_LTC/C6 renamed /LTC/C6
- net /L_LTC/C7 renamed /LTC/C7
- net /L_LTC/C8 renamed /LTC/C8
- net /L_LTC/C9 renamed /LTC/C9
- net /L_LTC/VREG renamed /LTC/VREG
- net Net-(IC1-DRIVE) renamed /LTC/NPNB
- net Net-(Q1-C) renamed /LTC/NPNC
- C1 pad 1: /IN+ -> /IN-
- C1 pad 2: /ICL+ -> /ICL-
- C2 pad 1: /IN- -> /IN+
- C2 pad 2: /ICL- -> /ICL+
- C3 pad 1: /OCL+ -> /OCL-
- C3 pad 2: /OUT+ -> /OUT-
- C4 pad 1: /OCL- -> /OCL+
- C4 pad 2: /OUT- -> /OUT+
- C6 pad 1: Net-(IC1-VREF2) -> /LTC/VREF2
- C7 pad 1: /L_LTC/VREF2 -> /LTC/VREF1
- IC1 pad 34: Net-(IC1-VREF2) -> /LTC/VREF2
- IC1 pad 35: /L_LTC/VREF2 -> /LTC/VREF1
- J1 pad 1: /IN+ -> /IN-
- J1 pad 2: /IN- -> /IN+
- J3 pad 1: /OUT- -> /OUT+
- J3 pad 2: /OUT+ -> /OUT-
- L1 pad 1: /ICL- -> /ICL+
- L1 pad 2: /IA- -> /IA+
- L1 pad 3: /IA+ -> /IA-
- L1 pad 4: /ICL+ -> /ICL-
- L2 pad 1: /IB- -> /IB+
- L2 pad 2: /OCL- -> /OCL+
- L2 pad 3: /OCL+ -> /OCL-
- L2 pad 4: /IB+ -> /IB-
- R33 pad 2: /L_LTC/VREF2 -> /LTC/VREF2
- R34 pad 2: /L_LTC/VREF2 -> /LTC/VREF2
- R35 pad 2: /L_LTC/VREF2 -> /LTC/VREF2
- R36 pad 2: /L_LTC/VREF2 -> /LTC/VREF2
- R8 pad 2: /L_LTC/VREF2 -> /LTC/VREF2
Routing:
- net /IB+: track 2.19 -> 63.2 mm, vias 0 -> 1
- net /IB-: track 2.19 -> 62.3 mm, vias 0 -> 1
- net /LTC/C10: track 2.90 -> 59.0 mm, vias 0 -> 2
- net /LTC/C11: track 2.90 -> 56.8 mm, vias 0 -> 2
- net /LTC/VREF2: track 0.00 -> 53.2 mm, vias 0 -> 5
- net /LTC/C12: track 2.90 -> 55.4 mm, vias 0 -> 2
- net /LTC/C7: track 2.90 -> 40.6 mm
- net /C12+: track 23.8 -> 60.5 mm, vias 4 -> 6
- net /LTC/C8: track 2.90 -> 34.3 mm
- net /IA-: track 2.19 -> 32.8 mm, vias 0 -> 1
- net /IA+: track 2.19 -> 32.0 mm, vias 0 -> 1
- net /LTC/C9: track 2.90 -> 27.9 mm
- net /C6+: track 4.40 -> 26.6 mm, vias 3 -> 4
- net /L_LTC/VREF2: track 10.4 -> 0.00 mm
- net /LTC/VREF1: track 0.00 -> 10.3 mm
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- added copper zone on F.Cu, net /LTC/VREG
Other:
- board text added: "IC"
- board text removed: "LTC"

Commit message: ltc rounting small fix
Parts:
- added G***: LOGO, Samacsys:PUTM_Logo_8mm, B.Cu at (211.8, 121.8)
Routing:
- net /LTC/C1: track 45.3 -> 47.1 mm
- net /LTC/C2: track 27.6 -> 28.1 mm

Commit message: bom update
Routing:
- net GND: vias 123 -> 122
Changed lines of the file:
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@@
-	)
-	(via
-		(at 144.9 124.7)
-		(size 0.45)
-		(drill 0.2)
-		(layers "F.Cu" "B.Cu")
-		(remove_unused_layers yes)
-		(keep_end_layers yes)
-		(free yes)
-		(zone_layer_connections "In1.Cu" "In2.Cu")
-		(net 62)
 	)
 	(via
@@
 			"727fcfd2-cb00-4e38-ade7-44ab4d5bf2f1" "7410a909-4c16-41c2-be8e-a0149837e18d"
 			"781a4f50-15db-40a9-a9f3-033613b2f9de" "7c58930e-8720-42c7-8f03-5b1bdbd404e6"
-			"80d8d6e9-290d-49da-b35f-2f785b3d6918" "861d230f-e262-4ff8-923b-ec551fcc63c3"
-			"8769c369-a4ee-4bcc-be1c-553ce618433d" "8a49fe9b-b4e5-44a2-8f90-d781facdadf6"
-			"8a98aa21-722c-41f3-a430-34dd8bee170b" "8ace75a3-aea9-4f4d-a710-1c291bed679f"
-			"8adb8766-ac71-4af9-9047-5acdce8ae124" "8b47554a-c4d8-4998-b7ac-9bbbacd5dec4"
-			"92036157-1afa-4c46-bb37-17bd0592bc1d" "93298f5e-9559-4bc6-af73-07af1d87d962"
-			"935a8066-ded2-4b99-8e25-062f51474e13" "938eba6a-421a-46e9-b7b7-bd77a833f41f"
-			"9473e1c0-9fb2-40d7-a552-8b69e0987b4f" "98bf36e9-ecb1-46ef-9807-c28d41f86bf5"
-			"9aa03bd7-daeb-463a-8fa0-ba9fc91b0a9e" "9c7ba603-edc7-4c94-a835-e883447fc5c3"
-			"9e92be09-bfe1-4028-b18d-30b41f92f348" "a1aba5d6-4aa9-4eea-bdb6-2167b5691a3c"
-			"a241c19c-f6b2-4e69-a601-c347ee13e6f2" "a4ce4b0d-8a4b-482e-842c-01451e47f6cd"
-			"aa96f543-f735-4814-ab9b-3ffa8c12871f" "aabcc406-57a2-4e81-a53d-a9fbb89994b9"
-			"ac9b9d9a-649f-4799-8423-095fd22c9118" "afb8e1ba-7000-4d6f-aa64-03ea68b09ab3"
-			"b0b966c2-83eb-448b-93ac-8be47fe3e6c0" "b1642c15-9ca6-44b1-8efd-2810192986f0"
-			"b19ae678-5c91-40f9-a180-747d60c29d33" "b3c7adcb-b692-4693-b6d1-331053d84d98"
-			"c03cf6d2-aaec-4493-8dc8-3d4952162b63" "c0f72584-499a-4674-8ac7-61b7612cdbcc"
-			"c1d97833-a679-449e-a117-f896228477f7" "c4fff7b8-8f0f-4826-9e64-8f7540177792"
-			"c56b0062-629c-448c-9456-90c86ed3dac2" "ca9b64dd-ab46-48fb-adf3-292a7bc7b302"
-			"cbf1a55b-4cc6-4482-8666-41cf909860e1" "cf0bd83d-aacb-4f63-a3ee-45690914072d"
-			"cf5b9b5b-edd3-4be3-b38b-bb165cc7ca21" "d1bd487e-e449-40a6-98f6-77d106d863d1"
-			"d222b0f2-0552-4c2d-a266-97411c179c32" "d36916e6-0097-4d9a-8808-c03b5fee7dd9"
-			"d4e32b29-4651-49b2-a116-20202cf0cff2" "d5e4987a-a27c-48b2-b63c-ff235d07a37a"
-			"daad7c60-3f4a-4e85-ab9d-cf523b605f5e" "daae7b82-c795-4dec-b977-ed60e7c662bc"
-			"dfb2bc31-a2f7-453f-aac9-63f426e6185f" "e0349030-582f-4c32-a74f-3e7477570319"
-			"e6a70113-6222-44ee-9f0d-34f8b25ed5de" "f07cf793-5894-49e2-96ca-44dee009ad7c"
-			"f3031a1f-7395-4611-8316-6ed6270acacd" "f3d578d6-339c-4d94-b807-719defad5437"
-			"fab1866c-26ef-4ee2-a985-905d81e87863" "fb9ec6a9-e67e-49ed-8c7f-8c064b5f5510"
-			"fbe77625-f452-4380-99a6-00071d265b41" "fd8e7db8-e0b6-472e-a041-f26db6520df5"
-			"fd94a7ab-212c-4950-93ed-6da316bb68bf" "ff8677de-4687-45f4-9c9d-b5ca52836d4f"
-		)
-	)
+			"861d230f-e262-4ff8-923b-ec551fcc63c3" "8769c369-a4ee-4bcc-be1c-553ce618433d"
+			"8a49fe9b-b4e5-44a2-8f90-d781facdadf6" "8a98aa21-722c-41f3-a430-34dd8bee170b"
+			"8ace75a3-aea9-4f4d-a710-1c291bed679f" "8adb8766-ac71-4af9-9047-5acdce8ae124"
+			"8b47554a-c4d8-4998-b7ac-9bbbacd5dec4" "92036157-1afa-4c46-bb37-17bd0592bc1d"
+			"93298f5e-9559-4bc6-af73-07af1d87d962" "935a8066-ded2-4b99-8e25-062f51474e13"
+			"938eba6a-421a-46e9-b7b7-bd77a833f41f" "9473e1c0-9fb2-40d7-a552-8b69e0987b4f"
+			"98bf36e9-ecb1-46ef-9807-c28d41f86bf5" "9aa03bd7-daeb-463a-8fa0-ba9fc91b0a9e"
+			"9c7ba603-edc7-4c94-a835-e883447fc5c3" "9e92be09-bfe1-4028-b18d-30b41f92f348"
+			"a1aba5d6-4aa9-4eea-bdb6-2167b5691a3c" "a241c19c-f6b2-4e69-a601-c347ee13e6f2"
+			"a4ce4b0d-8a4b-482e-842c-01451e47f6cd" "aa96f543-f735-4814-ab9b-3ffa8c12871f"
+			"aabcc406-57a2-4e81-a53d-a9fbb89994b9" "ac9b9d9a-649f-4799-8423-095fd22c9118"
+			"afb8e1ba-7000-4d6f-aa64-03ea68b09ab3" "b0b966c2-83eb-448b-93ac-8be47fe3e6c0"
+			"b1642c15-9ca6-44b1-8efd-2810192986f0" "b19ae678-5c91-40f9-a180-747d60c29d33"
+			"b3c7adcb-b692-4693-b6d1-331053d84d98" "c03cf6d2-aaec-4493-8dc8-3d4952162b63"
+			"c0f72584-499a-4674-8ac7-61b7612cdbcc" "c1d97833-a679-449e-a117-f896228477f7"
+			"c4fff7b8-8f0f-4826-9e64-8f7540177792" "c56b0062-629c-448c-9456-90c86ed3dac2"
+			"ca9b64dd-ab46-48fb-adf3-292a7bc7b302" "cbf1a55b-4cc6-4482-8666-41cf909860e1"
+			"cf0bd83d-aacb-4f63-a3ee-45690914072d" "cf5b9b5b-edd3-4be3-b38b-bb165cc7ca21"
+			"d1bd487e-e449-40a6-98f6-77d106d863d1" "d222b0f2-0552-4c2d-a266-97411c179c32"
+			"d36916e6-0097-4d9a-8808-c03b5fee7dd9" "d4e32b29-4651-49b2-a116-20202cf0cff2"
+			"d5e4987a-a27c-48b2-b63c-ff235d07a37a" "daad7c60-3f4a-4e85-ab9d-cf523b605f5e"
+			"daae7b82-c795-4dec-b977-ed60e7c662bc" "dfb2bc31-a2f7-453f-aac9-63f426e6185f"
+			"e0349030-582f-4c32-a74f-3e7477570319" "e6a70113-6222-44ee-9f0d-34f8b25ed5de"
+			"f07cf793-5894-49e2-96ca-44dee009ad7c" "f3031a1f-7395-4611-8316-6ed6270acacd"
+			"f3d578d6-339c-4d94-b807-719defad5437" "fab1866c-26ef-4ee2-a985-905d81e87863"
+			"fb9ec6a9-e67e-49ed-8c7f-8c064b5f5510" "fbe77625-f452-4380-99a6-00071d265b41"
+			"fd8e7db8-e0b6-472e-a041-f26db6520df5" "fd94a7ab-212c-4950-93ed-6da316bb68bf"
+			"ff8677de-4687-45f4-9c9d-b5ca52836d4f"
+		)
+	)
