File: hardware/Discharge.kicad_sch (KiCad schematic)
At the start: 3 parts

Commit message: new balancing schematic
Parts:
- R11: renamed from R17; value 100/1W -> 51/2W
- renumbered D3 to D11, R18 to R15
Connections:
- net C: now also R11.2; no longer R11.1
- net S renamed CO
- net CO: now also R11.1; no longer R11.2
Other:
- moved on the sheet: D11, R11, R15

Commit message: sync
Parts:
- R16: renamed from R11; footprint Resistor_SMD:R_1210_3225Metric -> Resistor_SMD:R_1206_3216Metric; Manufacturer_Part_Number CR2512-JW-680ELF -> (none); Mouser Part Number 652-CR2512-JW-680ELF -> (none); Mouser Price/Stock https://www.mouser.pl/ProductDetail/Bourns/CR2512-JW-680ELF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 -> (none)
- renumbered D11 to D4
Connections:
- net C renamed C_{IN}
- net CO renamed C_{VB}
Changed lines of the file:
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@@
 		)
 	)
-	(hierarchical_label "C"
+	(hierarchical_label "C_{IN}"
 		(shape input)
 		(at 128.27 97.79 180)
@@
 		)
 	)
-	(hierarchical_label "CO"
+	(hierarchical_label "C_{VB}"
 		(shape input)
 		(at 151.13 97.79 0)
@@
 		(pin "2"
 		)
-		(instances)
+		(instances
+			(project "PUTM_EV_AMS_SLAVE_2025"
+				(path "/532b753f-9344-4418-8e40-ab07f8ade533/6a830281-1331-4b0f-b6b7-336a24ad47cd/0e164975-552b-41db-ab4c-15ee9ada9cae"
+					(reference "R15")
+					(unit 1)
+				)
+				(path "/532b753f-9344-4418-8e40-ab07f8ade533/6a830281-1331-4b0f-b6b7-336a24ad47cd/0f62669b-9cdd-4694-9bfb-59ec24066851"
+					(reference "R19")
+					(unit 1)
+				)
+				(path "/532b753f-9344-4418-8e40-ab07f8ade533/6a830281-1331-4b0f-b6b7-336a24ad47cd/3aad698c-dd9c-4b44-8e14-130741fcaac0"
+					(reference "R23")
+					(unit 1)
+				)
+				(path "/532b753f-9344-4418-8e40-ab07f8ade533/6a830281-1331-4b0f-b6b7-336a24ad47cd/487a2533-b412-4f25-8904-c71ab49d0b98"
+					(reference "R31")
+					(unit 1)
+				)
+				(path "/532b753f-9344-4418-8e40-ab07f8ade533/6a830281-1331-4b0f-b6b7-336a24ad47cd/5aac5d05-8994-478a-8640-609643a8cd2a"
+					(reference "R13")
+					(unit 1)
+				)
+				(path "/532b753f-9344-4418-8e40-ab07f8ade533/6a830281-1331-4b0f-b6b7-336a24ad47cd/7776e438-044e-4a2f-bd02-61ad1a3bdd92"
+					(reference "R9")
+					(unit 1)
+				)
+				(path "/532b753f-9344-4418-8e40-ab07f8ade533/6a830281-1331-4b0f-b6b7-336a24ad47cd/7e63fd25-aa57-4409-a006-9fbd325dd5b9"
+					(reference "R29")
+					(unit 1)
+				)
+				(path "/532b753f-9344-4418-8e40-ab07f8ade533/6a830281-1331-4b0f-b6b7-336a24ad47cd/aeb95217-ca74-46f8-af72-c5bfa7f07f94"
+					(reference "R11")
+					(unit 1)
+				)
+				(path "/532b753f-9344-4418-8e40-ab07f8ade533/6a830281-1331-4b0f-b6b7-336a24ad47cd/bcbf3399-1a13-4b96-a068-729a5f43f0a3"
+					(reference "R27")
+					(unit 1)
+				)
+				(path "/532b753f-9344-4418-8e40-ab07f8ade533/6a830281-1331-4b0f-b6b7-336a24ad47cd/d8c5f666-1aa4-4889-8890-59f0f76439c6"
+					(reference "R21")
+					(unit 1)
+				)
+				(path "/532b753f-9344-4418-8e40-ab07f8ade533/6a830281-1331-4b0f-b6b7-336a24ad47cd/e4c47c00-c63c-4af0-8f1e-1f8ce04f8338"
+					(reference "R25")
+					(unit 1)
+				)
+				(path "/532b753f-9344-4418-8e40-ab07f8ade533/6a830281-1331-4b0f-b6b7-336a24ad47cd/e7334c2e-953a-46dd-9201-952cec0aa831"
+					(reference "R17")
+					(unit 1)
+				)
+			)
+		)
 	)
 	(symbol
@@
 		(on_board yes)
 		(dnp no)
-		(property "Reference" "R11"
+		(property "Reference" "R16"
 			(at 139.7 92.71 90)
 			(effects
@@
 			)
 		)
-		(property "Footprint" "Resistor_SMD:R_1210_3225Metric"
+		(property "Footprint" "Resistor_SMD:R_1206_3216Metric"
 			(at 139.7 97.79 0)
 			(effects
@@
 			)
 		)
-		(property "Manufacturer_Part_Number" "CR2512-JW-680ELF"
-			(at 139.7 97.79 0)
-			(effects
-				(font
-					(size 1.27 1.27)
-				)
-				(hide yes)
-			)
-		)
-		(property "Mouser Part Number" "652-CR2512-JW-680ELF"
-			(at 139.7 97.79 0)
-			(effects
-				(font
-					(size 1.27 1.27)
-				)
-				(hide yes)
-			)
-		)
-		(property "Mouser Price/Stock" "https://www.mouser.pl/ProductDetail/Bourns/CR2512-JW-680ELF?qs=sGAEpiMZZMvdGkrng054t3VembYjER8wDs7RjV0k1vk%3D"
+		(property "Manufacturer_Part_Number" ""
+			(at 139.7 97.79 0)
+			(effects
+				(font
+					(size 1.27 1.27)
+				)
+				(hide yes)
+			)
+		)
+		(property "Mouser Part Number" ""
+			(at 139.7 97.79 0)
+			(effects
+				(font
+					(size 1.27 1.27)
+				)
+				(hide yes)
+			)
+		)
+		(property "Mouser Price/Stock" ""
 			(at 139.7 97.79 0)
 			(effects
@@
 		(pin "2"
 		)
-		(instances)
+		(instances
+			(project "PUTM_EV_AMS_SLAVE_2025"
+				(path "/532b753f-9344-4418-8e40-ab07f8ade533/6a830281-1331-4b0f-b6b7-336a24ad47cd/0e164975-552b-41db-ab4c-15ee9ada9cae"
+					(reference "R16")
+					(unit 1)
+				)
+				(path "/532b753f-9344-4418-8e40-ab07f8ade533/6a830281-1331-4b0f-b6b7-336a24ad47cd/0f62669b-9cdd-4694-9bfb-59ec24066851"
+					(reference "R20")
+					(unit 1)
+				)
+				(path "/532b753f-9344-4418-8e40-ab07f8ade533/6a830281-1331-4b0f-b6b7-336a24ad47cd/3aad698c-dd9c-4b44-8e14-130741fcaac0"
+					(reference "R24")
+					(unit 1)
+				)
+				(path "/532b753f-9344-4418-8e40-ab07f8ade533/6a830281-1331-4b0f-b6b7-336a24ad47cd/487a2533-b412-4f25-8904-c71ab49d0b98"
+					(reference "R32")
+					(unit 1)
+				)
+				(path "/532b753f-9344-4418-8e40-ab07f8ade533/6a830281-1331-4b0f-b6b7-336a24ad47cd/5aac5d05-8994-478a-8640-609643a8cd2a"
+					(reference "R14")
+					(unit 1)
+				)
+				(path "/532b753f-9344-4418-8e40-ab07f8ade533/6a830281-1331-4b0f-b6b7-336a24ad47cd/7776e438-044e-4a2f-bd02-61ad1a3bdd92"
+					(reference "R10")
+					(unit 1)
+				)
+				(path "/532b753f-9344-4418-8e40-ab07f8ade533/6a830281-1331-4b0f-b6b7-336a24ad47cd/7e63fd25-aa57-4409-a006-9fbd325dd5b9"
+					(reference "R30")
+					(unit 1)
+				)
+				(path "/532b753f-9344-4418-8e40-ab07f8ade533/6a830281-1331-4b0f-b6b7-336a24ad47cd/aeb95217-ca74-46f8-af72-c5bfa7f07f94"
+					(reference "R12")
+					(unit 1)
+				)
+				(path "/532b753f-9344-4418-8e40-ab07f8ade533/6a830281-1331-4b0f-b6b7-336a24ad47cd/bcbf3399-1a13-4b96-a068-729a5f43f0a3"
+					(reference "R28")
+					(unit 1)
+				)
+				(path "/532b753f-9344-4418-8e40-ab07f8ade533/6a830281-1331-4b0f-b6b7-336a24ad47cd/d8c5f666-1aa4-4889-8890-59f0f76439c6"
+					(reference "R22")
+					(unit 1)
+				)
+				(path "/532b753f-9344-4418-8e40-ab07f8ade533/6a830281-1331-4b0f-b6b7-336a24ad47cd/e4c47c00-c63c-4af0-8f1e-1f8ce04f8338"
+					(reference "R26")
+					(unit 1)
+				)
+				(path "/532b753f-9344-4418-8e40-ab07f8ade533/6a830281-1331-4b0f-b6b7-336a24ad47cd/e7334c2e-953a-46dd-9201-952cec0aa831"
+					(reference "R18")
+					(unit 1)
+				)
+			)
+		)
 	)
 	(symbol
@@
 		(on_board yes)
 		(dnp no)
-		(property "Reference" "D11"
+		(property "Reference" "D4"
 			(at 143.51 104.14 0)
 			(effects
@@
 		(pin "2"
 		)
-		(instances)
+		(instances
+			(project "PUTM_EV_AMS_SLAVE_2025"
+				(path "/532b753f-9344-4418-8e40-ab07f8ade533/6a830281-1331-4b0f-b6b7-336a24ad47cd/0e164975-552b-41db-ab4c-15ee9ada9cae"
+					(reference "D4")
+					(unit 1)
+				)
+				(path "/532b753f-9344-4418-8e40-ab07f8ade533/6a830281-1331-4b0f-b6b7-336a24ad47cd/0f62669b-9cdd-4694-9bfb-59ec24066851"
+					(reference "D6")
+					(unit 1)
+				)
+				(path "/532b753f-9344-4418-8e40-ab07f8ade533/6a830281-1331-4b0f-b6b7-336a24ad47cd/3aad698c-dd9c-4b44-8e14-130741fcaac0"
+					(reference "D8")
+					(unit 1)
+				)
+				(path "/532b753f-9344-4418-8e40-ab07f8ade533/6a830281-1331-4b0f-b6b7-336a24ad47cd/487a2533-b412-4f25-8904-c71ab49d0b98"
+					(reference "D12")
+					(unit 1)
+				)
+				(path "/532b753f-9344-4418-8e40-ab07f8ade533/6a830281-1331-4b0f-b6b7-336a24ad47cd/5aac5d05-8994-478a-8640-609643a8cd2a"
+					(reference "D3")
+					(unit 1)
+				)
+				(path "/532b753f-9344-4418-8e40-ab07f8ade533/6a830281-1331-4b0f-b6b7-336a24ad47cd/7776e438-044e-4a2f-bd02-61ad1a3bdd92"
+					(reference "D1")
+					(unit 1)
+				)
+				(path "/532b753f-9344-4418-8e40-ab07f8ade533/6a830281-1331-4b0f-b6b7-336a24ad47cd/7e63fd25-aa57-4409-a006-9fbd325dd5b9"
+					(reference "D11")
+					(unit 1)
+				)
+				(path "/532b753f-9344-4418-8e40-ab07f8ade533/6a830281-1331-4b0f-b6b7-336a24ad47cd/aeb95217-ca74-46f8-af72-c5bfa7f07f94"
+					(reference "D2")
+					(unit 1)
+				)
+				(path "/532b753f-9344-4418-8e40-ab07f8ade533/6a830281-1331-4b0f-b6b7-336a24ad47cd/bcbf3399-1a13-4b96-a068-729a5f43f0a3"
+					(reference "D10")
+					(unit 1)
+				)
+				(path "/532b753f-9344-4418-8e40-ab07f8ade533/6a830281-1331-4b0f-b6b7-336a24ad47cd/d8c5f666-1aa4-4889-8890-59f0f76439c6"
+					(reference "D7")
+					(unit 1)
+				)
+				(path "/532b753f-9344-4418-8e40-ab07f8ade533/6a830281-1331-4b0f-b6b7-336a24ad47cd/e4c47c00-c63c-4af0-8f1e-1f8ce04f8338"
+					(reference "D9")
+					(unit 1)
+				)
+				(path "/532b753f-9344-4418-8e40-ab07f8ade533/6a830281-1331-4b0f-b6b7-336a24ad47cd/e7334c2e-953a-46dd-9201-952cec0aa831"
+					(reference "D5")
+					(unit 1)
+				)
+			)
+		)
 	)
 )
