File: hardware/Ltc.kicad_sch (KiCad schematic)
At the start: 15 parts, among them CN7 4x100nF, IC1 LTC6804HG-1#PBF

Commit message: sync
Parts:
- removed C?: 100nF, Capacitor_SMD:C_0603_1608Metric, symbol PUTM_EV_BMS_HV_Slave_2021-rescue:C_Small-Device
- removed CN7: 4x100nF, Resistor_SMD:R_Array_Convex_4x0603, symbol ca064x104k4racauto:CA064X104K4RACAUTO
- added R1, R2: 120, Resistor_SMD:R_0603_1608Metric, symbol PUTM_EV_BMS_HV_Slave_2021-rescue:R_Small-Device
- added R3: 51/2W, Resistor_SMD:R_1206_3216Metric, symbol PUTM_EV_BMS_HV_Slave_2021-rescue:R_Small-Device
- renumbered C19 to C5, C18 to C9, R7 to R5, R8 to R6, R5 to R7, R2 to R8, RN7 to RN1
Connections:
- net C1+: no longer IC1.24 (C1)
- net C10+: no longer IC1.6 (C10)
- net C11+: no longer IC1.4 (C11)
- net C12+: no longer IC1.2 (C12)
- net C2+: no longer IC1.22 (C2)
- net C3+: no longer IC1.20 (C3)
- net C4+: no longer IC1.18 (C4)
- net C5+: no longer IC1.16 (C5)
- net C6+: no longer IC1.14 (C6)
- net C7+: no longer IC1.12 (C7)
- net C8+: no longer IC1.10 (C8)
- net C9+: no longer IC1.8 (C9)
- net IMA: now also R2.1
- net IMB: now also R1.1
- net IPA: now also R2.2
- net IPB: now also R1.2
- net V-: no longer C9.2, C?.2, C?.2, C?.2, IC1.26 (C0), IC1.30 (V-), IC1.31 (V-), IC1.36 (SWTEN), R6.2
- net S1 renamed C1
- net C1: now also IC1.24 (C1)
- net S10 renamed C10
- net C10: now also IC1.6 (C10)
- net S11 renamed C11
- net C11: now also IC1.4 (C11)
- net S12 renamed C12
- net C12: now also IC1.2 (C12)
- net S2 renamed C2
- net C2: now also IC1.22 (C2)
- net S3 renamed C3
- net C3: now also IC1.20 (C3)
- net S4 renamed C4
- net C4: now also IC1.18 (C4)
- net S5 renamed C5
- net C5: now also IC1.16 (C5)
- net S6 renamed C6
- net C6: now also IC1.14 (C6)
- net S7 renamed C7
- net C7: now also IC1.12 (C7)
- net S8 renamed C8
- net C8: now also IC1.10 (C8)
- net S9 renamed C9
- net C9: now also IC1.8 (C9)
- new net C0: IC1.26 (C0), R3.1
- new net C1-: R3.2
- new net GND: C9.2, C?.2, C?.2, C?.2, IC1.30 (V-), IC1.31 (V-), IC1.36 (SWTEN), R6.2
Other:
- added sheet DCH10 (Discharge.kicad_sch)
- added sheet DCH11 (Discharge.kicad_sch)
- added sheet DCH12 (Discharge.kicad_sch)
- added sheet DCH2 (Discharge.kicad_sch)
- added sheet DCH3 (Discharge.kicad_sch)
- added sheet DCH4 (Discharge.kicad_sch)
- added sheet DCH5 (Discharge.kicad_sch)
- added sheet DCH6 (Discharge.kicad_sch)
- added sheet DCH7 (Discharge.kicad_sch)
- added sheet DCH8 (Discharge.kicad_sch)
- added sheet DCH9 (Discharge.kicad_sch)
- sheet DCH1 ports: added C_{IN}, C_{VB}; removed none
- note removed: "CELL/TEMP DISCONN"
- note removed: "sprawdzic jeszcze tego sipa"
- moved on the sheet: C9, C?, Q?, R5, R6, R7
