File: hardware/Ltc.kicad_sch (KiCad schematic)
At the start: 19 parts, among them IC1 LTC6804HG-1#PBF

Commit message: done
Connections:
- net VREF2: now also C?.1, IC1.34 (VREF2); no longer C?.1, IC1.35 (VREF1)
- net NPNC: now reaches C9.1, Q?.2 (C), R7.2
- net NPNB: now reaches IC1.38 (DRIVE), Q?.1 (B)
- new net VREF1: C?.1, IC1.35 (VREF1)
Changed lines of the file:
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@@
+		(color 0 0 0 0)
+	)
+	(junction
+		(at 181.61 143.51)
+		(diameter 0)
 		(color 0 0 0 0)
 	)
@@
 		(pts
 			(xy 80.01 110.49) (xy 143.51 110.49)
+		)
+		(stroke
+			(width 0)
+			(type default)
+		)
+	)
+	(wire
+		(pts
+			(xy 181.61 143.51) (xy 193.04 143.51)
 		)
 		(stroke
@@
 		)
 	)
+	(label "NPNB"
+		(at 186.69 100.33 180)
+		(fields_autoplaced yes)
+		(effects
+			(font
+				(size 0.685 0.685)
+			)
+			(justify right bottom)
+		)
+	)
 	(label "C11"
 		(at 140.97 57.15 180)
@@
 		)
 	)
-	(label "VREF2"
+	(label "VREF1"
 		(at 193.04 140.97 0)
 		(fields_autoplaced yes)
@@
 		)
 	)
+	(label "NPNC"
+		(at 196.85 92.71 0)
+		(fields_autoplaced yes)
+		(effects
+			(font
+				(size 0.685 0.685)
+			)
+			(justify left bottom)
+		)
+	)
 	(label "C9"
 		(at 140.97 72.39 180)
@@
 		)
 	)
+	(label "VREF2"
+		(at 193.04 143.51 0)
+		(fields_autoplaced yes)
+		(effects
+			(font
+				(size 1.27 1.27)
+			)
+			(justify left bottom)
+		)
+	)

Commit message: bom update
Parts:
- R1, R2, R33, R34, R35, R36, R4, R5, R6, R7, R8: Mouser Part Number (none) -> --
- R3: value 51/2W -> 51/>1W; Mouser Part Number (none) -> 754-HRG3216P51R0DT1; Mouser Price/Stock (none) -> https://www.mouser.pl/ProductDetail/Susumu/HRG3216P-51R0-D-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
