File: hardware/PUTM_EV_AMS_SLAVE_2025.kicad_sch (KiCad schematic)
At the start: 7 parts, among them J1 M80-5100442, J2 TST-110-01-T-D, J3 M80-5100442

Commit message: rounting + layout
Parts:
- added L1, L2: 100-500uH, Inductor_SMD:L_CommonModeChoke_Coilcraft_1812CAN, symbol Device:L_Coupled_Small_1243
Connections:
- net IA+: now also L1.3; no longer C1.2
- net IA-: now also L1.2; no longer C2.2
- net IB+: now also L2.4; no longer C3.1
- net IB-: now also L2.1; no longer C4.1
- new net ICL+: C1.2, L1.4
- new net ICL-: C2.2, L1.1
- new net OCL+: C3.1, L2.3
- new net OCL-: C4.1, L2.2
Other:
- moved on the sheet: J2

Commit message: done
Connections:
- net IA+: now also L1.2; no longer L1.3
- net IA-: now also L1.3; no longer L1.2
- net IB+: now also L2.1; no longer L2.4
- net IB-: now also L2.4; no longer L2.1
- net ICL+: now also C2.2, L1.1; no longer C1.2, L1.4
- net ICL-: now also C1.2, L1.4; no longer C2.2, L1.1
- net IN+: now also C2.1, J1.2 (Pin_2); no longer C1.1, J1.1 (Pin_1)
- net IN-: now also C1.1, J1.1 (Pin_1); no longer C2.1, J1.2 (Pin_2)
- net OCL+: now also C4.1, L2.2; no longer C3.1, L2.3
- net OCL-: now also C3.1, L2.3; no longer C4.1, L2.2
- net OUT+: now also C4.2, J3.1 (Pin_1); no longer C3.2, J3.2 (Pin_2)
- net OUT-: now also C3.2, J3.2 (Pin_2); no longer C4.2, J3.1 (Pin_1)
Other:
- sheet L_LTC renamed LTC
- moved on the sheet: C1, C2, C3, C4, J1

Commit message: bom update
Parts:
- J2: value TST-110-01-T-D -> IDC20
- L1, L2: Mouser Part Number (none) -> 673-PE-1812AGC101STS
Changed lines of the file:
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@@
+			)
+		)
+		(property "Arrow Part Number" ""
+			(at 214.63 91.44 0)
+			(effects
+				(font
+					(size 1.27 1.27)
+				)
+				(hide yes)
+			)
+		)
+		(property "Arrow Price/Stock" ""
+			(at 214.63 91.44 0)
+			(effects
+				(font
+					(size 1.27 1.27)
+				)
+				(hide yes)
+			)
+		)
+		(property "Mouser Url" ""
+			(at 214.63 91.44 0)
+			(effects
+				(font
+					(size 1.27 1.27)
+				)
+				(hide yes)
 			)
 		)
@@
 			)
 		)
+		(property "Arrow Part Number" ""
+			(at 233.68 95.25 0)
+			(effects
+				(font
+					(size 1.27 1.27)
+				)
+				(hide yes)
+			)
+		)
+		(property "Arrow Price/Stock" ""
+			(at 233.68 95.25 0)
+			(effects
+				(font
+					(size 1.27 1.27)
+				)
+				(hide yes)
+			)
+		)
+		(property "Mouser Url" ""
+			(at 233.68 95.25 0)
+			(effects
+				(font
+					(size 1.27 1.27)
+				)
+				(hide yes)
+			)
+		)
 		(pin "2"
 		)
@@
 			)
 		)
+		(property "Arrow Part Number" ""
+			(at 81.28 91.44 0)
+			(effects
+				(font
+					(size 1.27 1.27)
+				)
+				(hide yes)
+			)
+		)
+		(property "Arrow Price/Stock" ""
+			(at 81.28 91.44 0)
+			(effects
+				(font
+					(size 1.27 1.27)
+				)
+				(hide yes)
+			)
+		)
+		(property "Mouser Url" ""
+			(at 81.28 91.44 0)
+			(effects
+				(font
+					(size 1.27 1.27)
+				)
+				(hide yes)
+			)
+		)
 		(pin "2"
 		)
@@
 			)
 		)
-		(property "TME Electronic Components Part Number" ""
+		(property "Arrow Part Number" ""
 			(at 96.52 95.25 0)
 			(effects
@@
 			)
 		)
-		(property "TME Electronic Components Price/Stock" ""
+		(property "Arrow Price/Stock" ""
+			(at 96.52 95.25 0)
+			(effects
+				(font
+					(size 1.27 1.27)
+				)
+				(hide yes)
+			)
+		)
+		(property "Mouser Part Number" "673-PE-1812AGC101STS"
+			(at 96.52 95.25 0)
+			(effects
+				(font
+					(size 1.27 1.27)
+				)
+				(hide yes)
+			)
+		)
+		(property "Mouser Url" ""
 			(at 96.52 95.25 0)
 			(effects
@@
 			)
 		)
+		(property "Arrow Part Number" ""
+			(at 64.77 95.25 0)
+			(effects
+				(font
+					(size 1.27 1.27)
+				)
+				(hide yes)
+			)
+		)
+		(property "Arrow Price/Stock" ""
+			(at 64.77 95.25 0)
+			(effects
+				(font
+					(size 1.27 1.27)
+				)
+				(hide yes)
+			)
+		)
+		(property "Mouser Url" ""
+			(at 64.77 95.25 0)
+			(effects
+				(font
+					(size 1.27 1.27)
+				)
+				(hide yes)
+			)
+		)
 		(pin "2"
 		)
@@
 			)
 		)
+		(property "Arrow Part Number" ""
+			(at 81.28 99.06 0)
+			(effects
+				(font
+					(size 1.27 1.27)
+				)
+				(hide yes)
+			)
+		)
+		(property "Arrow Price/Stock" ""
+			(at 81.28 99.06 0)
+			(effects
+				(font
+					(size 1.27 1.27)
+				)
+				(hide yes)
+			)
+		)
+		(property "Mouser Url" ""
+			(at 81.28 99.06 0)
+			(effects
+				(font
+					(size 1.27 1.27)
+				)
+				(hide yes)
+			)
+		)
 		(pin "2"
 		)
@@
 			)
 		)
-		(property "TME Electronic Components Part Number" ""
+		(property "Arrow Part Number" ""
 			(at 199.39 95.25 0)
 			(effects
@@
 			)
 		)
-		(property "TME Electronic Components Price/Stock" ""
+		(property "Arrow Price/Stock" ""
+			(at 199.39 95.25 0)
+			(effects
+				(font
+					(size 1.27 1.27)
+				)
+				(hide yes)
+			)
+		)
+		(property "Mouser Part Number" "673-PE-1812AGC101STS"
+			(at 199.39 95.25 0)
+			(effects
+				(font
+					(size 1.27 1.27)
+				)
+				(hide yes)
+			)
+		)
+		(property "Mouser Url" ""
 			(at 199.39 95.25 0)
 			(effects
@@
 			)
 		)
+		(property "Arrow Part Number" ""
+			(at 214.63 99.06 0)
+			(effects
+				(font
+					(size 1.27 1.27)
+				)
+				(hide yes)
+			)
+		)
+		(property "Arrow Price/Stock" ""
+			(at 214.63 99.06 0)
+			(effects
+				(font
+					(size 1.27 1.27)
+				)
+				(hide yes)
+			)
+		)
+		(property "Mouser Url" ""
+			(at 214.63 99.06 0)
+			(effects
+				(font
+					(size 1.27 1.27)
+				)
+				(hide yes)
+			)
+		)
 		(pin "2"
 		)
@@
 			)
 		)
-		(property "Value" "TST-110-01-T-D"
+		(property "Value" "IDC20"
 			(at 148.59 29.21 0)
 			(effects
@@
 			(at 147.32 43.18 0)
 			(effects
+				(font
+					(size 1.27 1.27)
+				)
+				(hide yes)
+			)
+		)
+		(property "Arrow Part Number" ""
+			(at 147.32 43.18 0)
+			(effects
+				(font
+					(size 1.27 1.27)
+				)
+				(hide yes)
+			)
+		)
+		(property "Arrow Price/Stock" ""
+			(at 147.32 43.18 0)
+			(effects
+				(font
+					(size 1.27 1.27)
+				)
+				(hide yes)
+			)
+		)
+		(property "Mouser Url" ""
+			(at 147.32 43.18 0)
+			(effects

Commit message: bom update
Parts:
- J2: Manufacturer_Part_Number TST-110-01-T-D -> HTST11001TDV; Mouser Part Number 200-TST11001TD -> 200-HTST11001TDV
Changed lines of the file:
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@@
 			)
 		)
-		(property "Manufacturer_Part_Number" "TST-110-01-T-D"
+		(property "Manufacturer_Part_Number" "HTST11001TDV"
 			(at 147.32 43.18 0)
 			(effects
@@
 			)
 		)
-		(property "Mouser Part Number" "200-TST11001TD"
+		(property "Mouser Part Number" "200-HTST11001TDV"
 			(at 147.32 43.18 0)
 			(effects
