File: hardware/BQ79616.kicad_sch (KiCad schematic)
At the start: 30 parts, among them IC2 BQ79616PAPR, Q2 100V/2W

Commit message: bom update
Parts:
- C38: Mouser Part Number (none) -> 81-GRT188R72A103KE1J
- C39: Mouser Part Number (none) -> 963-H168SC7224KTCA1J
- C4, C41: Mouser Part Number (none) -> --
- C40, C42, C43, C44, C45: Mouser Part Number (none) -> 187-CL10B105KA8NNNL
- D17, D18: CBOM LL-S190SC-2S -> (none)
- Q2: Mouser Part Number (none) -> 522-FZT653TA
- R2, R61: value 510 -> 10k; Mouser Part Number 603-RT0603FRE07330RL -> --
- R50, R53, R54, R62, R63, R64, R65, R66, R67, R68, R69: Mouser Part Number 603-RT0603FRE07330RL -> --
- TH1, TH2: Mouser Part Number (none) -> 810-NTCGS163JF103FT7

Commit message: v2.0.1b
Connections:
- net CVDD: now also IC2.52 (RX)
- no-connect marks 5 -> 4

Commit message: dev-hard-v3.0
Parts:
- removed D17: LED, LED_SMD:LED_0603_1608Metric, symbol PUTM_EV_BMS_HV_Slave_2021-rescue:LED_Small_ALT-Device
- removed R2: 10k, Resistor_SMD:R_0603_1608Metric, symbol PUTM_EV_BMS_HV_Slave_2021-rescue:R_Small-Device
- removed TH1, TH2: 10k/β=?, Resistor_SMD:R_0603_1608Metric, symbol Device:Thermistor_NTC
- added C1, C10, C11, C12, C13, C18, C19, C2, C20, C21, C22, C23, C24, C25, C26, C27, C28, C29, C3, C5, C6, C7, C8, C9: 470nF/16V, Capacitor_SMD:C_0603_1608Metric, symbol Device:C_Small
- added Q1: 2N7002, Package_TO_SOT_SMD:SOT-23, symbol Transistor_FET:2N7002
- added R70: 100, Resistor_SMD:R_0603_1608Metric, symbol PUTM_EV_BMS_HV_Slave_2021-rescue:R_Small-Device
- R51: value 33/1W -> 10/3W; footprint Resistor_SMD:R_1206_3216Metric -> Resistor_SMD:R_2512_6332Metric; Manufacturer_Part_Number CR2512-JW-680ELF -> 352210RJT; Mouser Part Number 652-CR2512-JW-680ELF -> 279-352210RJT; Mouser Price/Stock https://www.mouser.pl/ProductDetail/Bourns/CR2512-JW-680ELF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 -> https://www.mouser.pl/ProductDetail/YAGEO/RT0603FRE07330RL?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
- R54: value 200 -> 100
- R61: value 10k -> 1k
Connections:
- net CB13 is gone; now on net BAT: IC2.8 (CB13)
- net CB14 is gone; now on net BAT: IC2.6 (CB14)
- net CB15 is gone; now on net BAT: IC2.4 (CB15)
- net CB16 is gone; now on net BAT: IC2.2 (CB16)
- net VC13 is gone; now on net BAT: IC2.9 (VC13)
- net VC14 is gone; now on net BAT: IC2.7 (VC14)
- net VC15 is gone; now on net BAT: IC2.5 (VC15)
- net VC16 is gone; now on net BAT: IC2.3 (VC16)
- net AUX2/TH8+: now also Q1.1 (G); no longer D18.1 (K)
- net C12+: now also R52.1, R70.1
- net CB0: now also C13.2
- net CB1: now also C12.2, C13.1
- net CB10: now also C2.2, C3.1
- net CB11: now also C1.2, C2.1
- net CB12: now also C1.1
- net CB2: now also C11.2, C12.1
- net CB3: now also C10.2, C11.1
- net CB4: now also C10.1, C9.2
- net CB5: now also C8.2, C9.1
- net CB6: now also C7.2, C8.1
- net CB7: now also C6.2, C7.1
- net CB8: now also C5.2, C6.1
- net CB9: now also C3.2, C5.1
- net GND: now also Q1.2 (S)
- net VC0: now also C29.2
- net VC1: now also C28.2, C29.1
- net VC10: now also C19.2, C20.1
- net VC11: now also C18.2, C19.1
- net VC12: now also C18.1
- net VC2: now also C27.2, C28.1
- net VC3: now also C26.2, C27.1
- net VC4: now also C25.2, C26.1
- net VC5: now also C24.2, C25.1
- net VC6: now also C23.2, C24.1
- net VC7: now also C22.2, C23.1
- net VC8: now also C21.2, C22.1
- net VC9: now also C20.2, C21.1
- net C16+: no longer names the net of R54.1
- net C16+: now also R70.2; no longer R52.1
- new net: D18.1 (K), Q1.3 (D)
Other:
- removed sheet DCH13
- removed sheet DCH14
- removed sheet DCH15
- removed sheet DCH16
- sheet DCH1 ports: added none; removed CB-, VC-
- sheet DCH10 ports: added none; removed CB-, VC-
- sheet DCH11 ports: added none; removed CB-, VC-
- sheet DCH12 ports: added none; removed CB-, VC-
- sheet DCH2 ports: added none; removed CB-, VC-
- sheet DCH3 ports: added none; removed CB-, VC-
- sheet DCH4 ports: added none; removed CB-, VC-
- sheet DCH5 ports: added none; removed CB-, VC-
- sheet DCH6 ports: added none; removed CB-, VC-
- sheet DCH7 ports: added none; removed CB-, VC-
- sheet DCH8 ports: added none; removed CB-, VC-
- sheet DCH9 ports: added none; removed CB-, VC-
- moved on the sheet: D18
