File: hardware/PUTM_EV_AMS_SLAVE.kicad_sch (KiCad schematic)
At the start: 19 parts, among them J1 M80-5020442, J2 M80-5020442, J6 522071060, J7 522071060, J8 522071060, T1 SM91502ALE, T2 SM91502ALE

Commit message: slight fixes
Other:
- note added: "CONN MEAS"
Changed lines of the file:
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@@
 	(paper "A4")
+	(rectangle
+		(start 86.36 15.24)
+		(end 208.28 69.85)
+		(stroke
+			(width 0)
+			(type dash)
+			(color 132 132 132 1)
+		)
+		(fill
+			(type none)
+		)
+	)
 	(rectangle
 		(start 181.61 73.66)
@@
 		(effects
 			(font
+				(size 2 2)
+				(thickness 1)
+				(bold yes)
+				(color 132 132 132 1)
+			)
+			(justify right bottom)
+		)
+	)
+	(text "CONN MEAS"
+		(exclude_from_sim no)
+		(at 207.01 68.58 0)
+		(effects
+			(font
